Commit message: Dev: update tinker models (urdf, stl, etc.)

File: bipedal_locomotion_isaaclab/exts/bipedal_locomotion/bipedal_locomotion/assets/tinker/urdf/h1 copy.urdf (robot description, URDF)
Before this commit: robot h1, 11 links, 10 joints
Joints:
- joint J_L0: limit lower=-0.3 upper=0.3 effort=12 velocity=20 -> lower=-0.7 upper=0.7 effort=12 velocity=20; origin xyz=0.0025357 0.053301 0.056145 rpy=0 0 0 -> xyz=-0.002787 0.053542 0.054381 rpy=0 0 0
- joint J_L1: limit lower=-0.2 upper=0.2 effort=20 velocity=20 -> lower=-0.38 upper=0.46 effort=20 velocity=20; origin xyz=-0.010958 0 -0.054965 rpy=0 0 0 -> xyz=0.016958 0 -0.053917 rpy=0 0 0
- joint J_L2: limit lower=-0.57 upper=1.57 effort=20 velocity=20 -> lower=-1.57 upper=1.57 effort=20 velocity=20; origin xyz=0.010958 0.073699 -0.014313 rpy=0 0 0 -> xyz=-0.012958 0.059001 -0.014313 rpy=0 0 0
- joint J_L3: limit lower=-2.35 upper=0.05 effort=20 velocity=20 -> lower=-2.35 upper=0.0 effort=20 velocity=20
- joint J_L4_ankle: limit lower=-0.6 upper=0.7 effort=12 velocity=20 -> lower=-1.2 upper=1.2 effort=12 velocity=20; origin xyz=0 0 -0.14149 rpy=0 0 0 -> xyz=0 0.025 -0.14049 rpy=0 0 0
- joint J_R0: limit lower=-0.3 upper=0.3 effort=12 velocity=20 -> lower=-0.7 upper=0.7 effort=12 velocity=20; origin xyz=0.0025357 -0.053425 0.056145 rpy=0 0 0 -> xyz=-0.002787 -0.053184 0.054381 rpy=0 0 0
- joint J_R1: limit lower=-0.2 upper=0.2 effort=20 velocity=20 -> lower=-0.38 upper=0.47 effort=20 velocity=20; origin xyz=-0.010958 0 -0.054965 rpy=0 0 0 -> xyz=0.016958 0 -0.053917 rpy=0 0 0
- joint J_R2: limit lower=-0.57 upper=1.57 effort=20 velocity=20 -> lower=-1.57 upper=1.57 effort=20 velocity=20; origin xyz=0.010958 -0.073575 -0.014313 rpy=0 0 0 -> xyz=-0.012958 -0.059 -0.014313 rpy=0 0 0
- joint J_R3: limit lower=-0.05 upper=2.35 effort=20 velocity=20 -> lower=0 upper=2.35 effort=20 velocity=20
- joint J_R4_ankle: limit lower=-0.7 upper=0.6 effort=12 velocity=20 -> lower=-1.2 upper=1.2 effort=12 velocity=20; origin xyz=0 0 -0.14149 rpy=0 0 0 -> xyz=0 -0.025 -0.14049 rpy=0 0 0
